Commit message: simple_armの可動範囲を変更

File: simple_arm/simple_arm_description/urdf/simple_arm.urdf (robot description, URDF)
Before this commit: robot simple_arm, 4 links, 3 joints
Joints:
- joint joint1: limit lower=-1.57 upper=1.57 effort=0 velocity=0 -> lower=-3.14 upper=3.14 effort=0 velocity=0
- joint joint2: limit lower=-1.57 upper=1.57 effort=0 velocity=0 -> lower=-3.14 upper=3.14 effort=0 velocity=0
